Commit message: add end effector frame

File: dynamixel_arm_description/urdf/dynamixel_arm.urdf (robot description, URDF)
Before this commit: robot dynamixel_arm, 12 links, 11 joints
Links:
- added link end_effector
Joints:
- added joint end_effector_frame: type fixed, parent link_5_1, child end_effector, origin xyz=0.0226 0.01194171505988 0.24098628193808 rpy=0 0 0

Commit message: edit gripper/motor ration

File: dynamixel_arm_description/urdf/dynamixel_arm.urdf (robot description, URDF)
Before this commit: robot dynamixel_arm, 13 links, 12 joints
Links:
- added link gripper_link
Joints:
- added joint outlink2: type revolute, parent link_5_1, child linkout_1_1, origin xyz=0.0313 -0.029351 0.106414 rpy=0 0 0, axis -1 0 0, limit lower=-0.575959 upper=0.383972 effort=100 velocity=100, mimic joint=gripper multiplier=0.05 offset=0.006
- joint gripper: axis -1 0 0 -> 0 0 1; child linkout_1_1 -> gripper_link; limit lower=-0.575959 upper=0.383972 effort=100 velocity=100 -> lower=-65.5269905 upper=94.98867187 effort=100 velocity=10.0; origin xyz=0.0313 -0.029351 0.106414 rpy=0 0 0 -> xyz=0.0226 0.01194171505988 0.24098628193808 rpy=0 0 0
- joint inlink1: mimic joint=gripper multiplier=-1.0 offset=0.0 -> joint=gripper multiplier=-0.05 offset=0.006
- joint inlink2: mimic joint=gripper multiplier=1.0 offset=0.0 -> joint=gripper multiplier=0.05 offset=0.006
- joint outlink1: mimic joint=gripper multiplier=-1.0 offset=0.0 -> joint=gripper multiplier=-0.05 offset=0.006
- joint outlink1_upper: mimic joint=gripper multiplier=-1.0 offset=0.0 -> joint=gripper multiplier=-0.05 offset=0.006
- joint outlink2_upper: mimic joint=gripper multiplier=1.0 offset=0.0 -> joint=gripper multiplier=0.05 offset=0.006

File: dynamixel_arm_description/urdf/dynamixel_arm_sim.urdf (robot description, URDF)
Before this commit: robot dynamixel_arm, 13 links, 12 joints
Links:
- added link gripper_link
Joints:
- added joint outlink2: type revolute, parent link_5_1, child linkout_1_1, origin xyz=0.0313 -0.029351 0.106414 rpy=0 0 0, axis -1 0 0, limit lower=-0.575959 upper=0.383972 effort=100 velocity=100, mimic joint=gripper multiplier=0.05 offset=0.006
- joint gripper: axis -1 0 0 -> 0 0 1; child linkout_1_1 -> gripper_link; limit lower=-0.575959 upper=0.383972 effort=100 velocity=100 -> lower=-65.5269905 upper=94.98867187 effort=100 velocity=10.0; origin xyz=0.0313 -0.029351 0.106414 rpy=0 0 0 -> xyz=0.0226 0.01194171505988 0.24098628193808 rpy=0 0 0
- joint inlink1: mimic joint=gripper multiplier=-1.0 offset=0.0 -> joint=gripper multiplier=-0.05 offset=0.006
- joint inlink2: mimic joint=gripper multiplier=1.0 offset=0.0 -> joint=gripper multiplier=0.05 offset=0.006
- joint outlink1: mimic joint=gripper multiplier=-1.0 offset=0.0 -> joint=gripper multiplier=-0.05 offset=0.006
- joint outlink1_upper: mimic joint=gripper multiplier=-1.0 offset=0.0 -> joint=gripper multiplier=-0.05 offset=0.006
- joint outlink2_upper: mimic joint=gripper multiplier=1.0 offset=0.0 -> joint=gripper multiplier=0.05 offset=0.006
